File: PCB/klor1_4.Single/klor1_4.kicad_pcb (KiCad board)
At the start: 2 copper layers, 160 x 118.2 mm, 88 parts, among them J1 MJ-4PP-9, J2 Haptic Buzz, J3 lv27, SW1 SW_PUSH-MX_W_LED, SW10 SW_PUSH-MX_W_LED, SW11 SW_PUSH-MX_W_LED, SW12 SW_PUSH-MX_W_LED, SW13 SW_PUSH-MX_W_LED, SW14 SW_PUSH-MX_W_LED, SW15 SW_PUSH-MX_W_LED, SW16 SW_PUSH-MX_W_LED, SW17 SW_PUSH-MX_W_LED, SW18 RotaryEncoder_Switch, SW19 SW_PUSH-MX_W_LED, SW2 SW_PUSH-MX_W_LED, SW20 SW_PUSH-MX_W_LED, SW21 SW_PUSH-MX_W_LED, SW22 SW_PUSH-MX_W_LED, SW3 SW_PUSH-MX_W_LED, SW4 SW_PUSH-MX_W_LED, SW5 SW_PUSH-MX_W_LED, SW6 SW_PUSH-MX_W_LED, SW7 SW_PUSH-MX_W_LED, SW8 SW_PUSH-MX_W_LED, SW9 SW_PUSH-MX_W_LED, U1 ProMicro

Commit message: single mcu
Parts:
- U1: value ProMicro -> ProMicro_Single; footprint KLOR:ProMicro -> KLOR:ProMicro_Single
- moved U1 0.79 mm to (98.4, 71.8)
Connections:
- U1 pad 1: LED -> (no net)
- U1 pad 10: row2 -> (no net)
- U1 pad 11: row3 -> (no net)
- U1 pad 12: AUDIO -> (no net)
- U1 pad 13: col5 -> (no net)
- U1 pad 14: col4 -> (no net)
- U1 pad 15: col3 -> (no net)
- U1 pad 16: col2 -> (no net)
- U1 pad 17: col1 -> (no net)
- U1 pad 18: col0 -> (no net)
- U1 pad 19: ENCB -> (no net)
- U1 pad 2: TX -> (no net)
- U1 pad 20: ENCA -> (no net)
- U1 pad 21: VCC -> (no net)
- U1 pad 22: RESET -> (no net)
- U1 pad 23: GND -> TX
- U1 pad 24: +BATT -> LED
- U1 pad 3: GND -> (no net)
- U1 pad 4: GND -> (no net)
- U1 pad 5: SDA -> (no net)
- U1 pad 6: SCL -> (no net)
- U1 pad 7: RX -> (no net)
- U1 pad 8: row0 -> (no net)
- U1 pad 9: row1 -> (no net)
Routing:
- net +BATT: track 32.9 -> 17.9 mm
- net LED: track 159.3 -> 172.8 mm
- net GND: track 202.0 -> 195.7 mm
- net TX: track 93.7 -> 92.2 mm

Commit message: single 2504151724
Parts:
- moved U1 0.62 mm to (98.3, 72.4)
Connections:
- U1 pad 1: (no net) -> +BATT
- U1 pad 10: (no net) -> col3
- U1 pad 11: (no net) -> col4
- U1 pad 12: (no net) -> col5
- U1 pad 13: (no net) -> AUDIO
- U1 pad 14: (no net) -> row3
- U1 pad 15: (no net) -> row2
- U1 pad 16: (no net) -> row1
- U1 pad 17: (no net) -> row0
- U1 pad 18: (no net) -> RX
- U1 pad 19: (no net) -> SCL
- U1 pad 2: (no net) -> GND
- U1 pad 20: (no net) -> SDA
- U1 pad 21: (no net) -> GND
- U1 pad 22: (no net) -> GND
- U1 pad 3: (no net) -> RESET
- U1 pad 4: (no net) -> VCC
- U1 pad 5: (no net) -> ENCA
- U1 pad 6: (no net) -> ENCB
- U1 pad 7: (no net) -> col0
- U1 pad 8: (no net) -> col1
- U1 pad 9: (no net) -> col2
Routing:
- net LED: track 172.8 -> 135.6 mm
- net row0: track 126.1 -> 109.0 mm
- net row3: track 168.6 -> 151.6 mm
- net col1: track 294.6 -> 278.8 mm
- net row1: track 176.3 -> 162.6 mm
- net row2: track 193.6 -> 179.9 mm
- net AUDIO: track 103.2 -> 89.5 mm
- net col5: track 141.9 -> 129.0 mm
- net col2: track 261.9 -> 249.0 mm
- net col3: track 255.3 -> 242.4 mm
- net col4: track 256.1 -> 244.9 mm
- net TX: track 92.2 -> 85.8 mm
- net +BATT: track 17.9 -> 13.7 mm
- net GND: track 195.7 -> 193.2 mm

Commit message: 202504152355
Routing:
- net col5: track 129.0 -> 48.2 mm
- net VCC: track 841.4 -> 790.3 mm, vias 25 -> 24
- net GND: track 193.2 -> 153.6 mm, vias 35 -> 34
- net SDA: track 279.5 -> 248.3 mm
- net col4: track 244.9 -> 214.3 mm, vias 10 -> 9
- net col0: track 241.8 -> 220.4 mm
- net SCL: track 260.6 -> 240.4 mm
- net RX: track 82.2 -> 62.9 mm
- net RESET: track 78.1 -> 59.5 mm, vias 2 -> 1
- net ENCB: track 65.9 -> 47.6 mm
- net ENCA: track 61.7 -> 43.8 mm
- net row2: track 179.9 -> 164.2 mm
- net Net-(D19-A): track 24.7 -> 9.07 mm, vias 1 -> 0
- net Net-(D17-A): track 29.4 -> 15.8 mm, vias 1 -> 0
- net Net-(D4-A): track 29.5 -> 16.0 mm, vias 1 -> 0
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Other:
- outline, holes or cut-outs redrawn

Commit message: 202504170029
Parts:
- removed JP1, JP2, JP3, JP4, JP5, JP6, JP7, JP8: Device_Jumper_NO_Small, Jumper:SolderJumper-2_P1.3mm_Open_TrianglePad1.0x1.5mm
Connections:
- OLED1 pad 1: Net-(OLED1-GND) -> GND
- OLED1 pad 2: Net-(OLED1-VCC) -> VCC
- OLED1 pad 3: Net-(OLED1-SCL) -> SCL
- OLED1 pad 4: Net-(OLED1-SDA) -> SDA
Routing:
- net col2: track 247.4 -> 173.2 mm, vias 8 -> 6
- net GND: track 153.6 -> 223.3 mm, vias 34 -> 32
- net col5: track 48.2 -> 82.4 mm, vias 4 -> 3
- net col3: track 240.0 -> 209.4 mm, vias 10 -> 8
- net col1: track 272.6 -> 258.3 mm, vias 7 -> 6
- net Net-(D21-A): track 24.3 -> 10.4 mm, vias 1 -> 0
- net Net-(D9-A): track 28.9 -> 15.6 mm, vias 1 -> 0
- net Net-(D8-A): track 29.6 -> 16.3 mm, vias 1 -> 0
- net col0: track 220.4 -> 207.3 mm, vias 4 -> 3
- net Net-(D20-A): track 21.5 -> 8.61 mm, vias 1 -> 0
- net Net-(SW11B-DOUT): track 30.5 -> 19.9 mm, vias 2 -> 0
- net Net-(SW2B-DOUT): track 29.9 -> 19.8 mm, vias 2 -> 0
- net Net-(SW4B-DOUT): track 38.9 -> 29.6 mm
- net Net-(SW15B-DIN): track 39.7 -> 30.7 mm
- net VCC: track 790.3 -> 781.5 mm, vias 24 -> 21
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
Commit message: 2504171658
Parts:
- removed JP12, JP14: VCC Jumper, Jumper:SolderJumper-2_P1.3mm_Open_TrianglePad1.0x1.5mm
- removed JP13, JP15: GND Jumper, Jumper:SolderJumper-2_P1.3mm_Open_TrianglePad1.0x1.5mm
- removed JP22, JP23, JP24, JP25, JP27, JP28: Device_Jumper_NO_Small, Jumper:SolderJumper-2_P1.3mm_Open_TrianglePad1.0x1.5mm
- moved D12 16.9 mm to (114.4, 101.5)
- moved D13 16.9 mm to (131.5, 104.4)
- moved D6 16.7 mm to (117.0, 82.5), turned to 180 degrees
- moved D7 13.1 mm to (131.6, 84.2), turned to 90 degrees
- moved D11 12.9 mm to (210.3, 96.8), turned to 80 degrees
- moved D2 12.6 mm to (131.2, 65.4), turned to 90 degrees
- moved D9 12.6 mm to (170.8, 85.3), turned to 86 degrees
- moved D16 12.5 mm to (187.9, 117.4), turned to 80 degrees
- moved D17 12.5 mm to (207.7, 115.8), turned to 80 degrees
- moved D15 12.5 mm to (170.5, 104.5), turned to 86 degrees
- moved D3 11.7 mm to (150.0, 57.5), turned to 90 degrees
- moved D1 10.8 mm to (112.6, 70.2), turned to 90 degrees
- moved D22 7.89 mm to (134.3, 125.3)
- moved D18 1.78 mm to (102.5, 106.3), turned to -90 degrees
Connections:
- BT1 pad 1: /PAD1 -> /PSW
- BT1 pad 2: /PAD2 -> GND
- J2 pad 1: Net-(J2-Pin_1) -> VCC
- J2 pad 2: Net-(J2-Pin_2) -> SDA
- J2 pad 5: Net-(J2-Pin_5) -> GND
Routing:
- net GND: track 223.3 -> 408.3 mm, vias 32 -> 28
- net VCC: track 781.5 -> 687.1 mm, vias 21 -> 23
- net col4: track 209.4 -> 128.8 mm, vias 6 -> 4
- net RX: track 62.9 -> 28.3 mm, vias 2 -> 1
- net Net-(D15-A): track 30.0 -> 0.00 mm, vias 1 -> 0
- net Net-(D11-A): track 33.3 -> 4.02 mm, vias 1 -> 0
- net row2: track 164.2 -> 193.0 mm, vias 1 -> 3
- net Net-(D7-A): track 30.5 -> 4.04 mm, vias 1 -> 0
- net col0: track 207.3 -> 184.9 mm, vias 3 -> 4
- net LED: track 120.6 -> 98.2 mm
- net row1: track 161.9 -> 140.9 mm, vias 1 -> 2
- net Net-(SW1B-DIN): track 29.9 -> 50.8 mm, vias 3 -> 0
- net Net-(SW15B-DIN): track 30.7 -> 47.2 mm
- net row3: track 136.8 -> 152.5 mm, vias 1 -> 3
- net col5: track 82.4 -> 67.0 mm, vias 3 -> 4
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
Commit message: 2504180105
Parts:
- removed JP16, JP17, JP18, JP19, JP20, JP21: Device_Jumper_NO_Small, Jumper:SolderJumper-2_P1.3mm_Open_TrianglePad1.0x1.5mm
- moved D13 1.68 mm to (132.4, 105.8)
Connections:
- J3 pad 2: Net-(J3-Pin_2) -> GND
- J3 pad 4: Net-(J3-Pin_4) -> SCL
- J3 pad 5: Net-(J3-Pin_5) -> SDA
Routing:
- net LED: track 98.2 -> 174.7 mm, vias 2 -> 4
- net col5: track 67.0 -> 116.9 mm, vias 4 -> 9
- net RX: track 28.3 -> 69.9 mm, vias 1 -> 3
- net col3: track 201.4 -> 237.7 mm
- net col4: track 128.8 -> 163.7 mm, vias 4 -> 8
- net col1: track 264.0 -> 231.2 mm
- net col0: track 184.9 -> 152.4 mm
- net col2: track 173.2 -> 204.8 mm, vias 6 -> 7
- net row1: track 140.9 -> 164.2 mm
- net VCC: track 687.1 -> 709.9 mm, vias 23 -> 24
- net SCL: track 231.4 -> 243.7 mm, vias 7 -> 8
- net row2: track 193.0 -> 186.4 mm, vias 3 -> 7
- net Net-(SW12B-DOUT): track 36.3 -> 31.5 mm
- net AUDIO: track 83.2 -> 87.8 mm, vias 0 -> 1
- net row3: track 152.5 -> 156.6 mm
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
Commit message: tümünü temizlemeden önce
Routing:
- net col1: track 231.2 -> 254.0 mm, vias 6 -> 7
- net col0: track 152.4 -> 174.8 mm, vias 4 -> 5
Other:
- outline, holes or cut-outs redrawn
Changed lines of the file:
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@@
 		)
 		(pad "" np_thru_hole circle
-			(at 3.81 -2.540005 176)
+			(at 3.81 -2.540006 176)
 			(size 3 3)
 			(drill 3)
@@
 		)
 		(pad "" np_thru_hole circle
-			(at 3.81 -2.540005 176)
+			(at 3.81 -2.540006 176)
 			(size 3 3)
 			(drill 3)
@@
 			(at -8.82 -7.15)
 			(size 1.524 1.524)
-			(drill 1)
+			(drill 0.8128)
 			(layers "*.Cu" "*.Mask")
 			(remove_unused_layers no)
@@
 		)
 		(pad "" np_thru_hole circle
-			(at 3.81 -2.540005 176)
+			(at 3.81 -2.540006 176)
 			(size 3 3)
 			(drill 3)
@@
 	(gr_line
 		(start 230.37422 93.128032)
-		(end 212.345 89.968273)
+		(end 212.319491 89.963802)
 		(stroke
 			(width 0.01)
@@
 	)
 	(gr_line
-		(start 212.319491 89.968273)
-		(end 214.014183 80.117575)
+		(start 212.319491 89.963802)
+		(end 214.014183 80.113104)
 		(stroke
 			(width 0.01)
@@
 	(gr_line
 		(start 205.345 129.32)
-		(end 223.470176 132.547258)
+		(end 223.322479 132.547258)
 		(stroke
 			(width 0.01)
@@
 	(via
 		(at 86.26 60.115)
-		(size 0.4)
-		(drill 0.3)
+		(size 0.8)
+		(drill 0.8)
 		(layers "F.Cu" "B.Cu")
 		(net 1)
@@
 	)
 	(segment
+		(start 94.965 89.2)
+		(end 90.235 93.93)
+		(width 1)
+		(layer "F.Cu")
+		(net 17)
+	)
+	(segment
 		(start 201.515 124.59)
 		(end 203.42181 122.68319)
@@
 	)
 	(segment
+		(start 94.965 84.29)
+		(end 94.965 89.2)
+		(width 1)
+		(layer "F.Cu")
+		(net 17)
+	)
+	(segment
 		(start 170.485 118.75)
 		(end 170.285 118.55)
@@
 	)
 	(via
+		(at 94.965 84.29)
+		(size 0.4)
+		(drill 0.3)
+		(layers "F.Cu" "B.Cu")
+		(net 17)
+	)
+	(via
 		(at 149.095 123.12)
 		(size 0.4)
@@
 	)
 	(segment
+		(start 94.965 80.86)
+		(end 94.965 84.29)
+		(width 1)
+		(layer "B.Cu")
+		(net 17)
+	)
+	(segment
 		(start 186.375 116.21)
 		(end 187.715 114.87)
@@
 	)
 	(segment
+		(start 89.475 75.37)
+		(end 94.965 80.86)
+		(width 1)
+		(layer "B.Cu")
+		(net 17)
+	)
+	(segment
 		(start 196.258345 80.768374)
 		(end 192.946423 84.080296)
@@
 	)
 	(segment
+		(start 94.965 84.29)
+		(end 94.965 84.31)
+		(width 1)
+		(layer "B.Cu")
+		(net 17)
+	)
+	(segment
 		(start 210.905 82.56)
 		(end 210.195 83.27)
@@
 	)
 	(segment
+		(start 88.285 91.91)
+		(end 88.285 93.53)
+		(width 1)
+		(layer "F.Cu")
+		(net 18)
+	)
+	(segment
 		(start 179.608302 117.575126)
 		(end 171.910126 117.575126)
@@
 	)
 	(via
+		(at 88.285 91.91)
+		(size 0.4)
+		(drill 0.3)
+		(layers "F.Cu" "B.Cu")
+		(net 18)
+	)
+	(via
 		(at 225.065 109.65)
 		(size 0.4)
@@
 	)
 	(segment
+		(start 86.884 75.421)
+		(end 86.884 90.509)
+		(width 1)
+		(layer "B.Cu")
+		(net 18)
+	)
+	(segment
 		(start 223.965 110.72)
 		(end 218.875 110.72)
 		(width 1)
 		(layer "B.Cu")
+		(net 18)
+	)
+	(segment
+		(start 86.884 90.509)
+		(end 88.285 91.91)
+		(width 1)
+		(layer "B.Cu")
+		(net 18)
+	)
+	(segment
+		(start 89.475 72.83)
+		(end 86.884 75.421)
+		(width 1)
+		(layer "B.Cu")
